File: ROBOTS/ROVER/Electric/FourCable/FourCable.kicad_sch (KiCad schematic)
At the start: 11 parts, among them J1 USB_B, M1 28BYJ-48, M2 28BYJ-48, M3 28BYJ-48, M4 28BYJ-48, U1 MCP23017_SP, U2 ULN2003, U3 ULN2003, U4 ULN2003, U5 ULN2003

Commit message: New Schema for Four Cable
Other:
- title: (none) -> Four Cable Slider
Changed lines of the file:
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@@
 	(generator_version "8.0")
 	(paper "A4")
+	(title_block
+		(title "Four Cable Slider")
+		(date "2025-01-08")
+		(rev "V1")
+	)
 	(junction
 		(at 224.79 100.33)
